Commit message: Fixed scene file

File: simulator_stack/kraken_visualization/kraken/scenes/scene_old.urdf (robot description, URDF)
Before this commit: robot scene, 11 links, 10 joints
Links:
- removed link gate_marker2
- removed link gate_marker3
- removed link gate_marker4
- removed link gate_marker5
- added link gate_marker; collision mesh filename=package://kraken_visualization/kraken/objects/marker.osg; visual mesh filename=package://kraken_visualization/kraken/objects/marker.osg
- link gate_L_rod: geometry collision mesh filename=package://kraken_visualization/kraken/objects/L_rod.osg; visual mesh filename=package://kraken_visualization/kraken/objects/L_rod.osg
- link gate_dropper: geometry collision mesh filename=package://kraken_visualization/kraken/objects/dropper.osg; visual mesh filename=package://kraken_visualization/kraken/objects/dropper.osg
- link gate_shooter: geometry collision mesh filename=package://kraken_visualization/kraken/objects/shooter.osg; visual mesh filename=package://kraken_visualization/kraken/objects/shooter.osg
Joints:
- removed joint gate_marker2_to_pool
- removed joint gate_marker3_to_pool
- removed joint gate_marker4_to_pool
- removed joint gate_marker5_to_pool
- added joint gate_marker_to_pool: type fixed, parent pool, child gate_marker, origin xyz=0 0 0 rpy=0 0 0.0
- joint gate_L_rod_to_pool: origin xyz=4.5 15 -1.1 rpy=0 3.14 0 -> xyz=8 8 0 rpy=0 0 0.0
- joint gate_buoy_blue_to_pool: origin xyz=7 8.16 0 rpy=0 0 0.0 -> xyz=3 3 0 rpy=0 0 0.0
- joint gate_buoy_green_to_pool: origin xyz=6.275 6.59 0 rpy=0 0 0.0 -> xyz=4 4 0 rpy=0 0 0.0
- joint gate_buoy_red_to_pool: origin xyz=5 6.84 0 rpy=0 0 0.0 -> xyz=5 5 0 rpy=0 0 0.0
- joint gate_dropper_to_pool: origin xyz=8.62 20.44 0 rpy=0 3.14 0.0 -> xyz=7 7 0 rpy=0 0 0.0
- joint gate_shooter_to_pool: origin xyz=3.36 21.95 0 rpy=4.71 0 0.4 -> xyz=6 6 0 rpy=0 0 0.0
