Commit message: Added new scene file

File: simulator_stack/kraken_visualization/kraken/scenes/scene.urdf (robot description, URDF)
Before this commit: robot scene, 8 links, 7 joints
Links:
- removed link gate_marker
- added link gate_marker2; collision mesh filename=package://auv_visulaization/kraken/objects/marker.osg; visual mesh filename=package://auv_visulaization/kraken/objects/marker.osg
- added link gate_marker3; collision mesh filename=package://auv_visulaization/kraken/objects/marker.osg; visual mesh filename=package://auv_visulaization/kraken/objects/marker.osg
- added link gate_marker4; collision mesh filename=package://auv_visulaization/kraken/objects/marker.osg; visual mesh filename=package://auv_visulaization/kraken/objects/marker.osg
- added link gate_marker5; collision mesh filename=package://auv_visulaization/kraken/objects/marker.osg; visual mesh filename=package://auv_visulaization/kraken/objects/marker.osg
- link gate_L_rod: geometry collision mesh filename=package://auv_visulaization/kraken/objects/L_rod.osg; visual mesh filename=package://auv_visulaization/kraken/objects/L_rod.osg
- link gate_buoy_blue: geometry collision mesh filename=package://auv_visulaization/kraken/objects/buoy_blue.osg; visual mesh filename=package://auv_visulaization/kraken/objects/buoy_blue.osg
- link gate_buoy_green: geometry collision mesh filename=package://auv_visulaization/kraken/objects/buoy_green.osg; visual mesh filename=package://auv_visulaization/kraken/objects/buoy_green.osg
- link gate_buoy_red: geometry collision mesh filename=package://auv_visulaization/kraken/objects/buoy_red.osg; visual mesh filename=package://auv_visulaization/kraken/objects/buoy_red.osg
- link gate_dropper: geometry collision mesh filename=package://auv_visulaization/kraken/objects/dropper.osg; visual mesh filename=package://auv_visulaization/kraken/objects/dropper.osg
- link gate_shooter: geometry collision mesh filename=package://auv_visulaization/kraken/objects/shooter.osg; visual mesh filename=package://auv_visulaization/kraken/objects/shooter.osg
- link pool: geometry collision mesh filename=package://auv_visulaization/kraken/terrain/pool.osg; visual mesh filename=package://auv_visulaization/kraken/terrain/pool.osg
Joints:
- removed joint gate_marker_to_pool
- removed joint gate_shooter_to_pool
- added joint gate_marker2_to_pool: type fixed, parent pool, child gate_marker2, origin xyz=8 3 0 rpy=0 0 1.9634
- added joint gate_marker3_to_pool: type fixed, parent pool, child gate_marker3, origin xyz=4.47 11.2 0 rpy=0 0 1.8
- added joint gate_marker4_to_pool: type fixed, parent pool, child gate_marker4, origin xyz=4 17 0 rpy=0 0 1.7
- added joint gate_marker5_to_pool: type fixed, parent pool, child gate_marker5, origin xyz=5 17 0 rpy=0 0 .76
- added joint gate_shoote5 sin(1.7-(pi/2))r_to_pool: type fixed, parent pool, child gate_shooter, origin xyz=3.36 21.95 0 rpy=0 0 0.0
- joint gate_L_rod_to_pool: origin xyz=8 8 0 rpy=0 0 0.0 -> xyz=4.5 15 0 rpy=0 0 0
- joint gate_buoy_blue_to_pool: origin xyz=3 3 0 rpy=0 0 0.0 -> xyz=7 8.16 0 rpy=0 0 0.0
- joint gate_buoy_green_to_pool: origin xyz=4 4 0 rpy=0 0 0.0 -> xyz=6.275 6.59 0 rpy=0 0 0.0
- joint gate_buoy_red_to_pool: origin xyz=5 5 0 rpy=0 0 0.0 -> xyz=5 6.84 0 rpy=0 0 0.0
- joint gate_dropper_to_pool: origin xyz=7 7 0 rpy=0 0 0.0 -> xyz=8.62 20.44 0 rpy=0 0 0.0

Commit message: Fixed arena

File: simulator_stack/kraken_visualization/kraken/scenes/scene.urdf (robot description, URDF)
Before this commit: robot scene, 11 links, 10 joints
Links:
- link gate_L_rod: geometry collision mesh filename=package://kraken_visualization/kraken/objects/gate.osg; visual mesh filename=package://kraken_visualization/kraken/objects/gate.osg
- link gate_buoy_blue: geometry collision mesh filename=package://kraken_visualization/kraken/objects/buoy_blue.osg; visual mesh filename=package://kraken_visualization/kraken/objects/buoy_blue.osg
- link gate_buoy_green: geometry collision mesh filename=package://kraken_visualization/kraken/objects/buoy_green.osg; visual mesh filename=package://kraken_visualization/kraken/objects/buoy_green.osg
- link gate_buoy_red: geometry collision mesh filename=package://kraken_visualization/kraken/objects/buoy_red.osg; visual mesh filename=package://kraken_visualization/kraken/objects/buoy_red.osg
- link gate_dropper: geometry collision mesh filename=package://kraken_visualization/kraken/objects/bins.osg; visual mesh filename=package://kraken_visualization/kraken/objects/bins.osg
- link gate_marker2: geometry collision mesh filename=package://kraken_visualization/kraken/objects/marker.osg; visual mesh filename=package://kraken_visualization/kraken/objects/marker.osg
- link gate_marker3: geometry collision mesh filename=package://kraken_visualization/kraken/objects/marker.osg; visual mesh filename=package://kraken_visualization/kraken/objects/marker.osg
- link gate_marker4: geometry collision mesh filename=package://kraken_visualization/kraken/objects/marker.osg; visual mesh filename=package://kraken_visualization/kraken/objects/marker.osg
- link gate_marker5: geometry collision mesh filename=package://kraken_visualization/kraken/objects/marker.osg; visual mesh filename=package://kraken_visualization/kraken/objects/marker.osg
- link gate_shooter: geometry collision mesh filename=package://kraken_visualization/kraken/objects/torp_board.osg; visual mesh filename=package://kraken_visualization/kraken/objects/torp_board.osg
- link pool: geometry collision mesh filename=package://kraken_visualization/kraken/terrain/pool.osg; visual mesh filename=package://kraken_visualization/kraken/terrain/pool.osg
Joints:
- removed joint gate_shoote5 sin(1.7-(pi/2))r_to_pool
- added joint gate_shooter_to_pool: type fixed, parent pool, child gate_shooter, origin xyz=3.36 21.95 0 rpy=4.71 0 0.4
- joint gate_L_rod_to_pool: origin xyz=4.5 15 0 rpy=0 0 0 -> xyz=4.5 15 -1.0 rpy=0 3.14 0
- joint gate_dropper_to_pool: origin xyz=8.62 20.44 0 rpy=0 0 0.0 -> xyz=8.62 20.44 0 rpy=0 3.14 0.0

Commit message: MOdified gitignore

File: simulator_stack/kraken_visualization/kraken/scenes/scene.urdf (robot description, URDF)
Before this commit: robot scene, 11 links, 10 joints
Links:
- link gate_L_rod: geometry collision mesh filename=package://kraken_visualization/kraken/objects/gate_obstacle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; visual mesh filename=package://kraken_visualization/kraken/objects/gate_obstacle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
- link gate_shooter: geometry collision mesh filename=package://kraken_visualization/kraken/objects/gate_obstacle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; visual mesh filename=package://kraken_visualization/kraken/objects/gate_obstacle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

Commit message: - Added 3d task object models spaceship(shoot) and gate to simulator scene.urdf - Modified marker_client and marker_server modules to work with simulator output - Removed *.dox from .gitignore and readding *.dox files

File: simulator_stack/kraken_visualization/kraken/scenes/scene.urdf (robot description, URDF)
Before this commit: robot scene, 11 links, 10 joints
Links:
- link gate_shooter: geometry collision mesh filename=package://kraken_visualization/kraken/objects/ship.osg; visual mesh filename=package://kraken_visualization/kraken/objects/ship.osg
Joints:
- joint gate_shooter_to_pool: origin xyz=3.36 21.95 0 rpy=4.71 0 0.4 -> xyz=3.36 21.95 0 rpy=6.28 0 0.4

Commit message: - Add updated 3d models to simulator - Change force scale in joystick control - Setting correct threshold values - Editing marker module to publish binary mono8 format output

File: simulator_stack/kraken_visualization/kraken/scenes/scene.urdf (robot description, URDF)
Before this commit: robot scene, 11 links, 10 joints
Links:
- link gate_shooter: geometry collision mesh filename=package://kraken_visualization/kraken/objects/shooter.osg; visual mesh filename=package://kraken_visualization/kraken/objects/shooter.osg
