Commit message: Added correceted simulation files

File: simulator_stack/kraken_visualization/kraken/scenes/kraken_stripped.urdf (robot description, URDF)
Before this commit: robot kraken, 11 links, 10 joints
Links:
- link base_link: geometry collision mesh filename=package://kraken_visualization/kraken/robot/new_model_krake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; visual mesh filename=package://kraken_visualization/kraken/robot/new_model_krake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

File: simulator_stack/kraken_visualization/kraken/scenes/scene.urdf (robot description, URDF)
Before this commit: robot scene, 8 links, 7 joints
Links:
- link gate_L_rod: geometry collision mesh filename=package://kraken_visualization/kraken/objects/L_rod.osg; visual mesh filename=package://kraken_visualization/kraken/objects/L_rod.osg
- link gate_buoy_blue: geometry collision mesh filename=package://kraken_visualization/kraken/objects/buoy_blue.osg; visual mesh filename=package://kraken_visualization/kraken/objects/buoy_blue.osg
- link gate_buoy_green: geometry collision mesh filename=package://kraken_visualization/kraken/objects/buoy_green.osg; visual mesh filename=package://kraken_visualization/kraken/objects/buoy_green.osg
- link gate_buoy_red: geometry collision mesh filename=package://kraken_visualization/kraken/objects/buoy_red.osg; visual mesh filename=package://kraken_visualization/kraken/objects/buoy_red.osg
- link gate_dropper: geometry collision mesh filename=package://kraken_visualization/kraken/objects/dropper.osg; visual mesh filename=package://kraken_visualization/kraken/objects/dropper.osg
- link gate_marker: geometry collision mesh filename=package://kraken_visualization/kraken/objects/marker.osg; visual mesh filename=package://kraken_visualization/kraken/objects/marker.osg
- link gate_shooter: geometry collision mesh filename=package://kraken_visualization/kraken/objects/shooter.osg; visual mesh filename=package://kraken_visualization/kraken/objects/shooter.osg
- link pool: geometry collision mesh filename=package://kraken_visualization/kraken/terrain/pool.osg; visual mesh filename=package://kraken_visualization/kraken/terrain/pool.osg

File: simulator_stack/kraken_visualization/kraken/scenes/test.urdf (robot description, URDF)
Before this commit: robot world_hi, 2 links, 1 joints
Links:
- link gate_marker: geometry collision mesh filename=/home/vinay/ros_workspace/ikat-auv-packages/kraken_visualiz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 scale=1.000000 1.000000 1.000000; visual mesh filename=/home/vinay/ros_workspace/ikat-auv-packages/kraken_visualiz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 scale=1.000000 1.000000 1.000000

Commit message: Added dvl sensor

File: simulator_stack/kraken_visualization/kraken/scenes/kraken_stripped.urdf (robot description, URDF)
Before this commit: robot kraken, 11 links, 10 joints
Links:
- added link dvl_link
Joints:
- added joint dvl_to_base_link: type fixed, parent base_link, child dvl_link, origin xyz=-0.602 0.00 -0.3 rpy=0 0 0, axis 0 0 1
